File: SM20/SM20.kicad_pcb (KiCad board)
At the start: 2 copper layers, 81 x 61.9 mm, 25 parts, among them U1 RP2040_Zero

Commit message: add nodes
Routing:
- net Row 0: track 0.00 -> 57.2 mm
- net Row 2: track 0.00 -> 57.0 mm
- net Row 1: track 0.00 -> 57.0 mm
- net Column 3: track 0.00 -> 38.1 mm
- net Column 2: track 0.00 -> 38.1 mm
- net Column 1: track 0.00 -> 38.1 mm
- net Column 0: track 0.00 -> 38.1 mm
- net Net-(D1-A): track 0.00 -> 7.88 mm
- net Net-(D2-A): track 0.00 -> 7.86 mm
- net Net-(D3-A): track 0.00 -> 7.84 mm
- net Net-(D5-A): track 0.00 -> 7.83 mm
- net Net-(D4-A): track 0.00 -> 7.82 mm
- net Net-(D6-A): track 0.00 -> 7.81 mm
- net Net-(D7-A): track 0.00 -> 7.79 mm
- net Net-(D9-A): track 0.00 -> 7.78 mm
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Changed lines of the file:
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@@
   (setup
     (pad_to_mask_clearance 0)
-    (grid_origin 107.315 20.955)
+    (grid_origin 21.59 20.955)
     (pcbplotparams
       (layerselection 0x00010fc_ffffffff)
@@
   (gr_line (start 19.20875 78.105) (end 19.20875 20.955)
     (stroke (width 0.1) (type default)) (layer "Edge.Cuts"))
+  (segment (start 91.44 36.255) (end 72.44 36.255) (width 0.25) (layer "B.Cu") (net 1))
+  (segment (start 72.44 36.255) (end 53.44 36.255) (width 0.25) (layer "B.Cu") (net 1))
+  (segment (start 34.66375 36.47875) (end 53.21625 36.47875) (width 0.25) (layer "B.Cu") (net 1))
+  (segment (start 53.21625 36.47875) (end 53.44 36.255) (width 0.25) (layer "B.Cu") (net 1))
+  (segment (start 34.44 36.255) (end 34.66375 36.47875) (width 0.25) (layer "B.Cu") (net 1))
+  (segment (start 34.44 26.185) (end 33.655 25.4) (width 0.25) (layer "B.Cu") (net 2))
+  (segment (start 34.44 32.955) (end 34.44 26.185) (width 0.25) (layer "B.Cu") (net 2))
+  (segment (start 53.44 32.955) (end 53.44 26.135) (width 0.25) (layer "B.Cu") (net 3))
+  (segment (start 53.44 26.135) (end 52.705 25.4) (width 0.25) (layer "B.Cu") (net 3))
+  (segment (start 72.44 32.955) (end 72.44 26.085) (width 0.25) (layer "B.Cu") (net 4))
+  (segment (start 72.44 26.085) (end 71.755 25.4) (width 0.25) (layer "B.Cu") (net 4))
+  (segment (start 91.44 26.035) (end 90.805 25.4) (width 0.25) (layer "B.Cu") (net 5))
+  (segment (start 91.44 32.955) (end 91.44 26.035) (width 0.25) (layer "B.Cu") (net 5))
+  (segment (start 53.44 55.255) (end 72.44 55.255) (width 0.25) (layer "B.Cu") (net 6))
+  (segment (start 53.44 55.255) (end 34.44 55.255) (width 0.25) (layer "B.Cu") (net 6))
+  (segment (start 91.44 55.255) (end 72.44 55.255) (width 0.25) (layer "B.Cu") (net 6))
+  (segment (start 53.44 51.955) (end 53.44 45.185) (width 0.25) (layer "B.Cu") (net 7))
+  (segment (start 53.44 45.185) (end 52.705 44.45) (width 0.25) (layer "B.Cu") (net 7))
+  (segment (start 72.44 51.955) (end 72.44 45.135) (width 0.25) (layer "B.Cu") (net 8))
+  (segment (start 72.44 45.135) (end 71.755 44.45) (width 0.25) (layer "B.Cu") (net 8))
+  (segment (start 91.44 45.085) (end 90.805 44.45) (width 0.25) (layer "B.Cu") (net 23))
+  (segment (start 91.44 51.955) (end 91.44 45.085) (width 0.25) (layer "B.Cu") (net 23))
+  (segment (start 34.44 70.955) (end 34.44 64.285) (width 0.25) (layer "B.Cu") (net 24))
+  (segment (start 34.44 64.285) (end 33.655 63.5) (width 0.25) (layer "B.Cu") (net 24))
+  (segment (start 72.44 74.255) (end 91.44 74.255) (width 0.25) (layer "B.Cu") (net 25))
+  (segment (start 53.44 74.255) (end 72.44 74.255) (width 0.25) (layer "B.Cu") (net 25))
+  (segment (start 34.44 74.255) (end 53.44 74.255) (width 0.25) (layer "B.Cu") (net 25))
+  (segment (start 72.44 70.955) (end 72.44 64.185) (width 0.25) (layer "B.Cu") (net 26))
+  (segment (start 72.44 64.185) (end 71.755 63.5) (width 0.25) (layer "B.Cu") (net 26))
+  (segment (start 91.44 70.955) (end 91.44 64.135) (width 0.25) (layer "B.Cu") (net 27))
+  (segment (start 91.44 64.135) (end 90.805 63.5) (width 0.25) (layer "B.Cu") (net 27))
+  (segment (start 27.305 46.99) (end 27.305 27.94) (width 0.25) (layer "F.Cu") (net 28))
+  (segment (start 27.305 46.99) (end 27.305 66.04) (width 0.25) (layer "F.Cu") (net 28))
+  (segment (start 46.355 66.04) (end 46.355 46.99) (width 0.25) (layer "F.Cu") (net 29))
+  (segment (start 46.355 27.94) (end 46.355 46.99) (width 0.25) (layer "F.Cu") (net 29))
+  (segment (start 65.405 66.04) (end 65.405 46.99) (width 0.25) (layer "F.Cu") (net 30))
+  (segment (start 65.405 46.99) (end 65.405 27.94) (width 0.25) (layer "F.Cu") (net 30))
+  (segment (start 84.455 46.99) (end 84.455 66.04) (width 0.25) (layer "F.Cu") (net 31))
+  (segment (start 84.455 27.94) (end 84.455 46.99) (width 0.25) (layer "F.Cu") (net 31))
+  (segment (start 34.44 45.235) (end 33.655 44.45) (width 0.25) (layer "B.Cu") (net 34))
+  (segment (start 34.44 51.955) (end 34.44 45.235) (width 0.25) (layer "B.Cu") (net 34))
+  (segment (start 53.44 70.955) (end 53.44 64.235) (width 0.25) (layer "B.Cu") (net 35))
+  (segment (start 53.44 64.235) (end 52.705 63.5) (width 0.25) (layer "B.Cu") (net 35))
 )

Commit message: finish
Routing:
- net Column 3: track 38.1 -> 104.9 mm, vias 0 -> 1
- net Row 2: track 57.0 -> 107.7 mm
- net Column 2: track 38.1 -> 86.9 mm, vias 0 -> 1
- net Row 1: track 57.0 -> 88.1 mm
- net Column 1: track 38.1 -> 63.1 mm
- net Row 0: track 57.2 -> 70.6 mm
- net Column 0: track 38.1 -> 48.8 mm
- added copper zone on B.Cu, net (none)
- added copper zone on F.Cu, net (none)
Changed lines of the file:
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@@
   (gr_line (start 19.20875 78.105) (end 19.20875 20.955)
     (stroke (width 0.1) (type default)) (layer "Edge.Cuts"))
+  (segment (start 23.495 30.32375) (end 26.19625 30.32375) (width 0.25) (layer "B.Cu") (net 1))
+  (segment (start 26.19625 30.32375) (end 32.1275 36.255) (width 0.25) (layer "B.Cu") (net 1))
+  (segment (start 32.1275 36.255) (end 34.44 36.255) (width 0.25) (layer "B.Cu") (net 1))
   (segment (start 91.44 36.255) (end 72.44 36.255) (width 0.25) (layer "B.Cu") (net 1))
   (segment (start 72.44 36.255) (end 53.44 36.255) (width 0.25) (layer "B.Cu") (net 1))
@@
   (segment (start 91.44 32.955) (end 91.44 26.035) (width 0.25) (layer "B.Cu") (net 5))
   (segment (start 53.44 55.255) (end 72.44 55.255) (width 0.25) (layer "B.Cu") (net 6))
+  (segment (start 24.57 33.93875) (end 24.57 52.51) (width 0.25) (layer "B.Cu") (net 6))
+  (segment (start 24.57 52.51) (end 27.315 55.255) (width 0.25) (layer "B.Cu") (net 6))
+  (segment (start 27.315 55.255) (end 34.44 55.255) (width 0.25) (layer "B.Cu") (net 6))
   (segment (start 53.44 55.255) (end 34.44 55.255) (width 0.25) (layer "B.Cu") (net 6))
+  (segment (start 23.495 32.86375) (end 24.57 33.93875) (width 0.25) (layer "B.Cu") (net 6))
   (segment (start 91.44 55.255) (end 72.44 55.255) (width 0.25) (layer "B.Cu") (net 6))
   (segment (start 53.44 51.955) (end 53.44 45.185) (width 0.25) (layer "B.Cu") (net 7))
@@
   (segment (start 34.44 70.955) (end 34.44 64.285) (width 0.25) (layer "B.Cu") (net 24))
   (segment (start 34.44 64.285) (end 33.655 63.5) (width 0.25) (layer "B.Cu") (net 24))
+  (segment (start 34.44 74.255) (end 24.88375 74.255) (width 0.25) (layer "B.Cu") (net 25))
   (segment (start 72.44 74.255) (end 91.44 74.255) (width 0.25) (layer "B.Cu") (net 25))
+  (segment (start 21.42 70.79125) (end 21.42 37.47875) (width 0.25) (layer "B.Cu") (net 25))
   (segment (start 53.44 74.255) (end 72.44 74.255) (width 0.25) (layer "B.Cu") (net 25))
   (segment (start 34.44 74.255) (end 53.44 74.255) (width 0.25) (layer "B.Cu") (net 25))
+  (segment (start 24.88375 74.255) (end 21.42 70.79125) (width 0.25) (layer "B.Cu") (net 25))
+  (segment (start 21.42 37.47875) (end 23.495 35.40375) (width 0.25) (layer "B.Cu") (net 25))
   (segment (start 72.44 70.955) (end 72.44 64.185) (width 0.25) (layer "B.Cu") (net 26))
   (segment (start 72.44 64.185) (end 71.755 63.5) (width 0.25) (layer "B.Cu") (net 26))
   (segment (start 91.44 70.955) (end 91.44 64.135) (width 0.25) (layer "B.Cu") (net 27))
   (segment (start 91.44 64.135) (end 90.805 63.5) (width 0.25) (layer "B.Cu") (net 27))
+  (segment (start 27.305 21.67) (end 25.79875 20.16375) (width 0.25) (layer "F.Cu") (net 28))
+  (segment (start 27.305 27.94) (end 27.305 21.67) (width 0.25) (layer "F.Cu") (net 28))
   (segment (start 27.305 46.99) (end 27.305 27.94) (width 0.25) (layer "F.Cu") (net 28))
+  (segment (start 25.79875 20.16375) (end 23.495 20.16375) (width 0.25) (layer "F.Cu") (net 28))
   (segment (start 27.305 46.99) (end 27.305 66.04) (width 0.25) (layer "F.Cu") (net 28))
   (segment (start 46.355 66.04) (end 46.355 46.99) (width 0.25) (layer "F.Cu") (net 29))
   (segment (start 46.355 27.94) (end 46.355 46.99) (width 0.25) (layer "F.Cu") (net 29))
+  (segment (start 24.57 23.77875) (end 42.19375 23.77875) (width 0.25) (layer "B.Cu") (net 29))
+  (segment (start 42.19375 23.77875) (end 46.355 27.94) (width 0.25) (layer "B.Cu") (net 29))
+  (segment (start 23.495 22.70375) (end 24.57 23.77875) (width 0.25) (layer "B.Cu") (net 29))
   (segment (start 65.405 66.04) (end 65.405 46.99) (width 0.25) (layer "F.Cu") (net 30))
+  (segment (start 62.87375 21.23875) (end 65.405 23.77) (width 0.25) (layer "F.Cu") (net 30))
+  (segment (start 28.59 24.955) (end 32.30625 21.23875) (width 0.25) (layer "F.Cu") (net 30))
+  (segment (start 65.405 23.77) (end 65.405 27.94) (width 0.25) (layer "F.Cu") (net 30))
   (segment (start 65.405 46.99) (end 65.405 27.94) (width 0.25) (layer "F.Cu") (net 30))
+  (segment (start 32.30625 21.23875) (end 62.87375 21.23875) (width 0.25) (layer "F.Cu") (net 30))
+  (via (at 28.59 24.955) (size 0.8) (drill 0.4) (layers "F.Cu" "B.Cu") (net 30))
+  (segment (start 23.78375 24.955) (end 28.59 24.955) (width 0.25) (layer "B.Cu") (net 30))
+  (segment (start 23.495 25.24375) (end 23.78375 24.955) (width 0.25) (layer "B.Cu") (net 30))
+  (segment (start 81.605 27.94) (end 74.59 34.955) (width 0.25) (layer "F.Cu") (net 31))
   (segment (start 84.455 46.99) (end 84.455 66.04) (width 0.25) (layer "F.Cu") (net 31))
+  (segment (start 84.455 27.94) (end 81.605 27.94) (width 0.25) (layer "F.Cu") (net 31))
   (segment (start 84.455 27.94) (end 84.455 46.99) (width 0.25) (layer "F.Cu") (net 31))
+  (segment (start 74.59 34.955) (end 67.59 34.955) (width 0.25) (layer "F.Cu") (net 31))
+  (via (at 67.59 34.955) (size 0.8) (drill 0.4) (layers "F.Cu" "B.Cu") (net 31))
+  (segment (start 30.463896 33.955) (end 24.292646 27.78375) (width 0.25) (layer "B.Cu") (net 31))
+  (segment (start 67.59 34.955) (end 44.59 34.955) (width 0.25) (layer "B.Cu") (net 31))
+  (segment (start 44.59 34.955) (end 43.59 33.955) (width 0.25) (layer "B.Cu") (net 31))
+  (segment (start 24.292646 27.78375) (end 23.495 27.78375) (width 0.25) (layer "B.Cu") (net 31))
+  (segment (start 43.59 33.955) (end 30.463896 33.955) (width 0.25) (layer "B.Cu") (net 31))
   (segment (start 34.44 45.235) (end 33.655 44.45) (width 0.25) (layer "B.Cu") (net 34))
   (segment (start 34.44 51.955) (end 34.44 45.235) (width 0.25) (layer "B.Cu") (net 34))
   (segment (start 53.44 70.955) (end 53.44 64.235) (width 0.25) (layer "B.Cu") (net 35))
   (segment (start 53.44 64.235) (end 52.705 63.5) (width 0.25) (layer "B.Cu") (net 35))
+  (zone (net 0) (net_name "") (layers "F&B.Cu") (hatch edge 0.5)
+    (connect_pads (clearance 0.5))
+    (min_thickness 0.25) (filled_areas_thickness no)
+    (fill yes (thermal_gap 0.5) (thermal_bridge_width 0.5) (island_removal_mode 1) (island_area_min 10))
+    (polygon
+      (pts
+        (xy 16.8275 16.1925)
+        (xy 102.5525 16.1925)
+        (xy 102.5525 82.8675)
+        (xy 16.8275 82.8675)
+      )
+    )
+  )
 )
